Commit message: Align front-leg URDF/IK and retune SoftTrot for taller, slower walk.
Fix front thigh/calf to 90/110 mm so sim matches IK, then retune SoftTrot
for less bounce, height 0.25, T=1.20 with the smaller 2.2/3.0 cm stride;
add --sim-parity patch inventory for A/B.

Co-authored-by: Cursor <cursoragent@cursor.com>

File: marsdog/urdf/marsdog.urdf (robot description, URDF)
Before this commit: robot marsdog, 53 links, 52 joints
Links:
- link fl_calf_link: geometry collision cylinder length=0.057 radius=0.023; collision cylinder length=0.065 radius=0.016
- link fl_thigh_roll_link: geometry collision box size=0.005 0.035 0.073; visual mesh filename=package://marsdog/meshes/fl_thigh_roll_link.STL
- link fr_calf_link: geometry collision cylinder length=0.057 radius=0.023; collision cylinder length=0.065 radius=0.016
- link fr_thigh_roll_link: geometry collision box size=0.005 0.035 0.073; visual mesh filename=package://marsdog/meshes/fr_thigh_roll_link.STL
Joints:
- joint fl_calf_joint: origin xyz=0.0235 0.0034955 -0.069995 rpy=0 0 0 -> xyz=0.02861305 0.00425604 -0.08522429 rpy=0 0 0
- joint fl_tarsus_joint: origin xyz=0.0040403 -0.0022336 -0.12194 rpy=0 0 0 -> xyz=0.003642077 -0.00201345 -0.1099213 rpy=0 0 0
- joint fr_calf_joint: origin xyz=0.02533 -0.0033053 -0.069363 rpy=0 0 0 -> xyz=0.03084125 -0.00402446 -0.08445485 rpy=0 0 0
- joint fr_tarsus_joint: origin xyz=0.0055464 0.0025664 -0.12187 rpy=0 0 0 -> xyz=0.004999904 0.002313528 -0.109862 rpy=0 0 0

Commit message: Pin SoftTrot to a single recipe SSOT and fix misleading defaults.
Merge NATURAL_SOFT_TROT_WBC/_REAL into one dict, align schema/GAIT/CLI help,
drop dead auto-trim patch inventory, and raise front tarsus URDF effort to 5 Nm.

Co-authored-by: Cursor <cursoragent@cursor.com>

File: marsdog/urdf/marsdog.urdf (robot description, URDF)
Before this commit: robot marsdog, 53 links, 52 joints
Joints:
- joint fl_tarsus_joint: limit lower=-0.03 upper=1.49 effort=0.4119 velocity=9.9484 -> lower=-0.03 upper=1.49 effort=5.0 velocity=9.9484
- joint fr_tarsus_joint: limit lower=-0.03 upper=1.49 effort=0.4119 velocity=9.9484 -> lower=-0.03 upper=1.49 effort=5.0 velocity=9.9484

Commit message: Hold Damiao at probed pose after enable; set front foot L3 to 63mm.
Bridge the probe/disable→enable MIT gap that thrashed tarsus during stand fade, keep URDF/IK/gravity_comp on the longer foot contact, and retune calf/waist gains.

Co-authored-by: Cursor <cursoragent@cursor.com>

File: marsdog/urdf/marsdog.urdf (robot description, URDF)
Before this commit: robot marsdog, 53 links, 52 joints
Links:
- link fl_tarsus_link: geometry collision cylinder length=0.063 radius=0.018; visual mesh filename=package://marsdog/meshes/fl_tarsus_link.STL
- link fr_tarsus_link: geometry collision cylinder length=0.063 radius=0.018; visual mesh filename=package://marsdog/meshes/fr_tarsus_link.STL
Joints:
- joint fl_foot_joint: origin xyz=0 -0.005449 -0.051948 rpy=0 0 0 -> xyz=0 -0.005449 -0.06276391 rpy=0 0 0
- joint fr_foot_joint: origin xyz=0 0.0055908 -0.051933 rpy=0 0 0 -> xyz=0 0.0055908 -0.06275144 rpy=0 0 0
